File: Main_circuit.kicad_sch (KiCad schematic)
At the start: 0 parts

Commit message: Ninth commit, power circuit
Other:
- sheet Capacitive Touch circuitry renamed Capacitive Touch Circuitry
- added sheet Voltage Sense Circuitry (V_sense_circuit.kicad_sch)
Changed lines of the file:
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@@
 	(paper "A4")
 	(sheet
-		(at 41.91 85.09)
-		(size 31.75 31.75)
+		(at 58.42 69.85)
+		(size 35.56 35.56)
 		(exclude_from_sim no)
 		(in_bom yes)
@@
 		)
 		(property "Sheetname" "Power Circuitry"
-			(at 41.91 84.3784 0)
+			(at 58.42 69.1384 0)
 			(show_name no)
 			(do_not_autoplace no)
@@
 		)
 		(property "Sheetfile" "Power_circuit.kicad_sch"
-			(at 41.91 117.4246 0)
+			(at 58.42 105.9946 0)
 			(show_name no)
 			(do_not_autoplace no)
@@
 	)
 	(sheet
-		(at 118.11 83.82)
+		(at 120.65 127)
+		(size 40.64 33.02)
+		(exclude_from_sim no)
+		(in_bom yes)
+		(on_board yes)
+		(dnp no)
+		(fields_autoplaced yes)
+		(stroke
+			(width 0.1524)
+			(type solid)
+		)
+		(fill
+			(color 0 0 0 0)
+		)
+		(property "Sheetname" "Voltage Sense Circuitry"
+			(at 120.65 126.2884 0)
+			(show_name no)
+			(do_not_autoplace no)
+			(effects
+				(font
+					(size 1.27 1.27)
+				)
+				(justify left bottom)
+			)
+		)
+		(property "Sheetfile" "V_sense_circuit.kicad_sch"
+			(at 120.65 160.6046 0)
+			(show_name no)
+			(do_not_autoplace no)
+			(effects
+				(font
+					(size 1.27 1.27)
+				)
+				(justify left top)
+			)
+		)
+		(instances
+			(project "Main_circuit"
+				(path "/02e8e4b0-2d68-453f-9f10-22ddb8bef6dd"
+					(page "5")
+				)
+			)
+		)
+	)
+	(sheet
+		(at 119.38 69.85)
 		(size 41.91 36.83)
 		(exclude_from_sim no)
@@
 		)
 		(property "Sheetname" "IC Circuitry"
-			(at 118.11 83.1084 0)
+			(at 119.38 69.1384 0)
 			(show_name no)
 			(do_not_autoplace no)
@@
 		)
 		(property "Sheetfile" "IC_circuit.kicad_sch"
-			(at 118.11 121.2346 0)
+			(at 119.38 107.2646 0)
 			(show_name no)
 			(do_not_autoplace no)
@@
 	)
 	(sheet
-		(at 200.66 96.52)
-		(size 22.86 20.32)
+		(at 189.23 71.12)
+		(size 35.56 35.56)
 		(exclude_from_sim no)
 		(in_bom yes)
@@
 			(color 0 0 0 0)
 		)
-		(property "Sheetname" "Capacitive Touch circuitry"
-			(at 200.66 95.8084 0)
+		(property "Sheetname" "Capacitive Touch Circuitry"
+			(at 189.23 70.4084 0)
 			(show_name no)
 			(do_not_autoplace no)
@@
 		)
 		(property "Sheetfile" "Cap_touch_circuit.kicad_sch"
-			(at 200.66 117.4246 0)
+			(at 189.23 107.2646 0)
 			(show_name no)
 			(do_not_autoplace no)
