File: Cap_touch_circuit.kicad_sch (KiCad schematic)
At the start: 0 parts

Commit message: Updated antenna and began work on touch circuitry
Parts:
- added Pad1: Touch Pad 1, symbol Connector_Generic:Conn_01x01
- added Pad2: Touch Pad 2, symbol Connector_Generic:Conn_01x01
- added Pad3: Touch Pad 3, symbol Connector_Generic:Conn_01x01
- added R6, R7: 4.7k, symbol Device:R
- added U2: CAP1203-1-SN, SOIC8_4P9X3P9MC_MCH, symbol 2026-10-18_22-41-59:CAP1203-1-SN
Connections:
- new net: Pad1.1 (Pin_1), U2.8 (CS1)
- new net: Pad2.1 (Pin_1), U2.7 (CS2)
- new net: Pad3.1 (Pin_1), U2.6 (CS3)
- new net +3.3V: R6.1, R7.1, U2.4 (VDD)
- new net GND: U2.1 (ALERT-), U2.5 (GND)
- new net Touch SCK: R7.2, U2.3 (SMCLK)
- new net Touch SDA: R6.2, U2.2 (SMDAT)
