File: V_sense_circuit.kicad_sch (KiCad schematic)
At the start: 0 parts

Commit message: Tenth commit, Voltage sense beginnings
Parts:
- added C15, C18, C19, C20, C21, C22, C23, C24: C, symbol Device:C
- added C16, C17: C_Po, symbol Device:C_Polarized
- added R10, R11, R12, R13, R8, R9: R, symbol Device:R
- added U3: ADE7953xCP, Package_CSP:LFCSP-28-1EP_5x5mm_P0.5mm_EP3.14x3.14mm, symbol Sensor:ADE7953xCP
Connections:
- new net: C15.1, C16.1, U3.3 (VINTD)
- new net: C21.2, R10.2, U3.6 (IAN)
- new net: C24.1, R13.1, U3.11 (VN)
- new net: C20.1, R9.2, U3.5 (IAP)
- new net: C19.2, R8.2, U3.2 (~{RESET})
- new net: C23.2, R12.2, U3.10 (IBN)
- new net: C17.1, C18.1, U3.15 (VINTA)
- new net: U3.7 (PULL_HIGH), U3.8 (PULL_HIGH)
- new net: C22.1, R11.2, U3.9 (IBP)
- new net +3.3V: C19.1, R8.1, U3.17 (VDD)
- new net GND: C15.2, C16.2, C17.2, C18.2, C20.2, C21.1, C22.2, C23.1, C24.2, R13.2
